File: KiCad/z80-cpu-mem.kicad_pcb (KiCad board)
At the start: 2 copper layers, 101.6 x 53.3 mm, 32 parts, among them J1 RCBus, SW1 RESET, U1 Z84C00-PLCC, U2 SST39SF040, U3 AS6C4008, U4 74AHCT174, U5 74AHCT138, U6 74AHCT32, U7 74AHCT32, U8 74AHCT00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

Commit message: Add files for v1.1
Signed-off-by: Sergey Kiselev <skiselev@gmail.com>
Parts:
- moved C4 10.2 mm to (179.1, 94.0)
- moved C6 10.2 mm to (179.1, 83.8)
- moved C5 10.2 mm to (128.3, 116.8)
- moved C8 10.2 mm to (128.3, 106.7)
Other:
- board text added: "Z80-CPM - Version 1.1 (C) 2025 Sergey Kiselev"
- board text removed: "Z80-CPM - Version 1.0 (C) 2025 Sergey Kiselev"
Changed lines of the file:
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@@
   (title_block
     (title "Z80-CPM: RCBus Z80 CPU and Memory Module")
-    (date "2025-05-21")
-    (rev "1.0")
+    (date "2025-06-28")
+    (rev "1.1")
     (company "Designed by Sergey Kiselev")
     (comment 2 "Licensed under CERN-OHL-S: https://cern-ohl.web.cern.ch")
@@
   )
   (footprint "My_Components:Cap_Cer_508" (layer "F.Cu")
-    (at 179.07 93.98 -90)
+    (at 179.07 83.82 -90)
     (descr "Ceramic Capacitor, 5.08mm lead spacing")
     (tags "Cap_Cer_508")
@@
   )
   (footprint "My_Components:Cap_Cer_508" (layer "F.Cu")
-    (at 128.27 106.68 -90)
+    (at 128.27 116.84 -90)
     (descr "Ceramic Capacitor, 5.08mm lead spacing")
     (tags "Cap_Cer_508")
@@
     (fp_line (start -2.413 1.651) (end -2.413 0.762) (layer "F.SilkS") (width 0.12))
     (fp_line (start 0 1.651) (end 0 1.651) (layer "F.SilkS") (width 0.12))
-    (fp_arc (start -2.285998 -0.762) (mid 0 -2.409654) (end 2.285999 -0.762) (layer "F.SilkS") (width 0.12))
+    (fp_arc (start -2.285998 -0.762) (mid 0.000001 -2.409655) (end 2.285999 -0.762) (layer "F.SilkS") (width 0.12))
     (fp_arc (start -2.285999 -0.762) (mid -1.40895 -1.954814) (end 0 -2.409655) (layer "F.SilkS") (width 0.12))
     (pad "1" thru_hole rect (at -2.54 0 90) (size 1.397 1.397) (drill 0.8128) (layers *.Cu *.Mask)
@@
       (effects (font (size 1 1) (thickness 0.15)))
     )
+    (fp_line (start 0.1778 2.4892) (end 1.651 1.016) (layer "F.SilkS") (width 0.12))
+    (fp_line (start 0 -2.5) (end 0 2.5) (layer "F.SilkS") (width 0.12))
+    (fp_line (start 1.016 -1.016) (end 1.7526 -1.7526) (layer "F.SilkS") (width 0.12))
+    (fp_line (start 2.032 -1.016) (end 2.032 1.016) (layer "F.SilkS") (width 0.12))
+    (fp_line (start 2.032 -1.016) (end 0 -1.016) (layer "F.SilkS") (width 0.12))
+    (fp_line (start 0 2.286) (end 1.27 1.016) (layer "F.SilkS") (width 0.12))
+    (fp_line (start 1.778 -1.016) (end 2.1082 -1.3462) (layer "F.SilkS") (width 0.12))
+    (fp_line (start 0.254 -1.016) (end 1.3335 -2.0955) (layer "F.SilkS") (width 0.12))
+    (fp_line (start 2.032 0.635) (end 2.4892 0.1778) (layer "F.SilkS") (width 0.12))
+    (fp_line (start 0 1.524) (end 0.508 1.016) (layer "F.SilkS") (width 0.12))
+    (fp_line (start 0.635 -1.016) (end 1.5494 -1.9304) (layer "F.SilkS") (width 0.12))
+    (fp_line (start 2.032 0.254) (end 2.4892 -0.2032) (layer "F.SilkS") (width 0.12))
+    (fp_line (start 0.635 2.413) (end 2.413 0.635) (layer "F.SilkS") (width 0.12))
+    (fp_line (start 2.032 -0.127) (end 2.4384 -0.5334) (layer "F.SilkS") (width 0.12))
+    (fp_line (start 2.032 1.016) (end 0 1.016) (layer "F.SilkS") (width 0.12))
+    (fp_line (start 0 -2.286) (end 0.2032 -2.4892) (layer "F.SilkS") (width 0.12))
+    (fp_line (start 1.397 -1.016) (end 1.9304 -1.5494) (layer "F.SilkS") (width 0.12))
+    (fp_line (start 0 -1.905) (end 0.5334 -2.4384) (layer "F.SilkS") (width 0.12))
+    (fp_line (start 0 1.905) (end 0.889 1.016) (layer "F.SilkS") (width 0.12))
+    (fp_line (start 2.032 -0.508) (end 2.3495 -0.8255) (layer "F.SilkS") (width 0.12))
+    (fp_line (start 0 -1.524) (end 0.8128 -2.3368) (layer "F.SilkS") (width 0.12))
+    (fp_line (start 1.2954 2.1336) (end 2.1336 1.2954) (layer "F.SilkS") (width 0.12))
+    (fp_line (start 0 -1.143) (end 1.0922 -2.2352) (layer "F.SilkS") (width 0.12))
+    (fp_line (start 2.032 -0.889) (end 2.2225 -1.0795) (layer "F.SilkS") (width 0.12))
     (fp_circle (center 0 0) (end 2.49936 0) (layer "F.SilkS") (width 0.12) (fill none))
     (pad "1" thru_hole rect (at -1.00076 0 270) (size 1.49098 1.49098) (drill 0.8001) (layers *.Cu *.Mask)
@@
   )
   (footprint "My_Components:Cap_Cer_508" (layer "F.Cu")
-    (at 128.27 116.84 -90)
+    (at 128.27 106.68 -90)
     (descr "Ceramic Capacitor, 5.08mm lead spacing")
     (tags "Cap_Cer_508")
@@
   )
   (footprint "My_Components:Cap_Cer_508" (layer "F.Cu")
-    (at 179.07 83.82 -90)
+    (at 179.07 93.98 -90)
     (descr "Ceramic Capacitor, 5.08mm lead spacing")
     (tags "Cap_Cer_508")
@@
   (gr_line (start 125.73 86.36) (end 133.35 78.74) (layer "Edge.Cuts") (width 0.05))
   (gr_line (start 227.33 80.01) (end 227.33 130.81) (layer "Edge.Cuts") (width 0.05))
-  (gr_text "Z80-CPM - Version 1.0\n(C) 2025 Sergey Kiselev" (at 193.675 95.5675) (layer "B.SilkS")
+  (gr_text "Z80-CPM - Version 1.1\n(C) 2025 Sergey Kiselev" (at 193.675 95.5675) (layer "B.SilkS")
     (effects (font (size 1 1) (thickness 0.15)) (justify mirror))
   )
@@
     (effects (font (size 1 1) (thickness 0.15)))
   )
-  (gr_text "Z80-CPM - Version 1.0\n(C) 2025 Sergey Kiselev" (at 153.035 117.1575 90) (layer "F.SilkS")
+  (gr_text "Z80-CPM - Version 1.1\n(C) 2025 Sergey Kiselev" (at 153.035 117.1575 90) (layer "F.SilkS")
     (effects (font (size 1 0.8) (thickness 0.15)) (justify left))
   )
